File: bq2423x-Breakout.kicad_pcb (KiCad board)
At the start: 2 copper layers, 26.5 x 23.9 mm, 18 parts, among them J1 Conn_01x09, J2 Conn_01x08, SW1 SW_DIP_x02, SW2 SW_DIP_x01, U1 bq24230

Commit message: Improve Silkscreen
Other:
- board text added: "↓BAT↓"
- board text added: "↓OUT↓"
- board text removed: "|BAT|"
- board text removed: "|OUT|"
