File: bq2423x-Breakout.sch (KiCad schematic (older format))
At the start: 2 parts, among them SW1 SW_DIP_x02, U1 bq24230

Commit message: Preliminary layout
Parts:
- added C1: 10µF 16V, Capacitor_SMD:C_0603_1608Metric, symbol Device:C_Small
- added C2: 10µF 10V, Capacitor_SMD:C_0603_1608Metric, symbol Device:C_Small
- added D1: LED_ABGR, LED_SMD:LED_Cree-PLCC4_2x2mm_CW, symbol local:LED_ABGR
- added J1: Conn_01x09, Connector_PinHeader_2.54mm:PinHeader_1x09_P2.54mm_Vertical, symbol Connector_Generic:Conn_01x09
- added J2: Conn_01x08, Connector_PinHeader_2.54mm:PinHeader_1x09_P2.54mm_Vertical, symbol Connector_Generic:Conn_01x09
- added R1: 1k8, Resistor_SMD:R_0603_1608Metric, symbol Device:R_Small
- added R2: 3k09, Resistor_SMD:R_0603_1608Metric, symbol Device:R_Small
- added RA1, RA2, RA3, RA4, RA5, RA6: 10k, Resistor_SMD:R_0603_1608Metric, symbol Device:R_Small
- added RV1: 30k, Potentiometer_SMD:Potentiometer_Bourns_TC33X_Vertical, symbol Device:R_POT
- added RV2: 4k7, Potentiometer_SMD:Potentiometer_Bourns_3314J_Vertical, symbol Device:R_POT
- added SW2: SW_DIP_x01, Button_Switch_SMD:SW_DIP_SPSTx01_Slide_Copal_CHS-01A_W5.08mm_P1.27mm_JPin, symbol Switch:SW_DIP_x01
- SW1: footprint (none) -> Button_Switch_SMD:SW_DIP_SPSTx02_Slide_Copal_CHS-02A_W5.08mm_P1.27mm_JPin; MPN (none) -> CHS-02TA; Manufacturer (none) -> Nidec Copal Electronics; Supplier:Digikey (none) -> 563-1005-1-ND
- U1: footprint (none) -> Package_DFN_QFN:QFN-16-1EP_3x3mm_P0.5mm_EP1.7x1.7mm_ThermalVias; MPN (none) -> BQ24230RGTR; Manufacturer (none) -> Texas Instruments; Supplier:Digikey (none) -> 296-23937-1-ND
Connections:
- net EN1: now also SW1.1, J1.2 (Pin_2), RA1.1
- net EN2: now also SW1.2, J1.3 (Pin_3), RA2.1
- net GND: now also C1.2, C2.2, J1.9 (Pin_9), J2.8 (Pin_8), J2.9 (Pin_9), R1.2, R2.2, RA1.2, RA2.2, RA3.1, RA4.2
- net OUT: now also C2.1, D1.1 (A), J2.1 (Pin_1), J2.2 (Pin_2)
- net TS: now reaches U1.1 (TS)
- net TS: now also J2.7 (Pin_7), SW2.1
- net ILIM: now reaches U1.12 (ILIM)
- net ILIM: now also J1.8 (Pin_8), RV2.2
- net IN: now reaches U1.13 (IN)
- net IN: now also SW1.3, SW1.4, C1.1, J1.1 (Pin_1)
- net TMR: now reaches U1.14 (TMR)
- net TMR: now also J1.7 (Pin_7)
- net ITERM: now reaches U1.15 (ITERM)
- net ITERM: now also J1.6 (Pin_6)
- net ISET: now reaches U1.16 (ISET)
- net ISET: now also J1.5 (Pin_5), RV1.2
- net BAT: now reaches U1.2 (BAT), U1.3 (BAT)
- net BAT: now also J2.5 (Pin_5), J2.6 (Pin_6)
- net ~CE: now reaches U1.4 (~CE)
- net ~CE: now also J1.4 (Pin_4), RA4.1
- net ~PGOOD: now reaches U1.7 (~PGOOD)
- net ~PGOOD: now also J2.3 (Pin_3), RA6.2
- net ~CHG: now reaches U1.9 (~CHG)
- net ~CHG: now also J2.4 (Pin_4), RA5.2
- new net: RA3.2, SW2.2
- new net: R2.1, RV2.1
- new net: R1.1, RV1.1
- new net: D1.3 (GK), RA6.1
- new net: D1.4 (RK), RA5.1
- no-connect marks 0 -> 3
Other:
- note removed: "- ENx Pulldown\n- SW1 nach OUT\n- Kondensatoren BAT\n- Kondensatoren IN\n- ~CE~ verbinden\n- 10k optional an TS\n- ILIM offen oder Poti?\n- Akkuverbinder?\n- ITERM nur auf Pin\n- ISET mit Poti?"
- moved on the sheet: SW1

Commit message: Fix MPN/etc. for RA*
Parts:
- RA1, RA2, RA3, RA4, RA5, RA6: MPN RC0603JR-071KL -> RC0603FR-0710KL; Supplier:Digikey 311-1.0KGRCT-ND -> 311-10.0KHRCT-ND
Changed lines of the file:
@@
 F 2 "Resistor_SMD:R_0603_1608Metric" H 4975 1650 50  0001 C CNN
 F 3 "~" H 4975 1650 50  0001 C CNN
-F 4 "RC0603JR-071KL" H 4975 1650 50  0001 C CNN "MPN"
+F 4 "RC0603FR-0710KL" H 4975 1650 50  0001 C CNN "MPN"
 F 5 "Yageo" H 4975 1650 50  0001 C CNN "Manufacturer"
-F 6 "311-1.0KGRCT-ND" H 4975 1650 50  0001 C CNN "Supplier:Digikey"
+F 6 "311-10.0KHRCT-ND" H 4975 1650 50  0001 C CNN "Supplier:Digikey"
 	1    4975 1650
 	1    0    0    -1
@@
 F 2 "Resistor_SMD:R_0603_1608Metric" H 5475 1650 50  0001 C CNN
 F 3 "~" H 5475 1650 50  0001 C CNN
-F 4 "RC0603JR-071KL" H 5475 1650 50  0001 C CNN "MPN"
+F 4 "RC0603FR-0710KL" H 5475 1650 50  0001 C CNN "MPN"
 F 5 "Yageo" H 5475 1650 50  0001 C CNN "Manufacturer"
-F 6 "311-1.0KGRCT-ND" H 5475 1650 50  0001 C CNN "Supplier:Digikey"
+F 6 "311-10.0KHRCT-ND" H 5475 1650 50  0001 C CNN "Supplier:Digikey"
 	1    5475 1650
 	1    0    0    -1
@@
 F 2 "Resistor_SMD:R_0603_1608Metric" H 5200 5300 50  0001 C CNN
 F 3 "~" H 5200 5300 50  0001 C CNN
-F 4 "RC0603JR-071KL" H 5200 5300 50  0001 C CNN "MPN"
+F 4 "RC0603FR-0710KL" H 5200 5300 50  0001 C CNN "MPN"
 F 5 "Yageo" H 5200 5300 50  0001 C CNN "Manufacturer"
-F 6 "311-1.0KGRCT-ND" H 5200 5300 50  0001 C CNN "Supplier:Digikey"
+F 6 "311-10.0KHRCT-ND" H 5200 5300 50  0001 C CNN "Supplier:Digikey"
 	1    5200 5300
 	-1   0    0    1
@@
 F 2 "Resistor_SMD:R_0603_1608Metric" H 5975 1650 50  0001 C CNN
 F 3 "~" H 5975 1650 50  0001 C CNN
-F 4 "RC0603JR-071KL" H 5975 1650 50  0001 C CNN "MPN"
+F 4 "RC0603FR-0710KL" H 5975 1650 50  0001 C CNN "MPN"
 F 5 "Yageo" H 5975 1650 50  0001 C CNN "Manufacturer"
-F 6 "311-1.0KGRCT-ND" H 5975 1650 50  0001 C CNN "Supplier:Digikey"
+F 6 "311-10.0KHRCT-ND" H 5975 1650 50  0001 C CNN "Supplier:Digikey"
 	1    5975 1650
 	1    0    0    -1
@@
 F 2 "Resistor_SMD:R_0603_1608Metric" H 7075 1625 50  0001 C CNN
 F 3 "~" H 7075 1625 50  0001 C CNN
-F 4 "RC0603JR-071KL" H 7075 1625 50  0001 C CNN "MPN"
+F 4 "RC0603FR-0710KL" H 7075 1625 50  0001 C CNN "MPN"
 F 5 "Yageo" H 7075 1625 50  0001 C CNN "Manufacturer"
-F 6 "311-1.0KGRCT-ND" H 7075 1625 50  0001 C CNN "Supplier:Digikey"
+F 6 "311-10.0KHRCT-ND" H 7075 1625 50  0001 C CNN "Supplier:Digikey"
 	1    7075 1625
 	0    1    1    0
@@
 F 2 "Resistor_SMD:R_0603_1608Metric" H 7075 1825 50  0001 C CNN
 F 3 "~" H 7075 1825 50  0001 C CNN
-F 4 "RC0603JR-071KL" H 7075 1825 50  0001 C CNN "MPN"
+F 4 "RC0603FR-0710KL" H 7075 1825 50  0001 C CNN "MPN"
 F 5 "Yageo" H 7075 1825 50  0001 C CNN "Manufacturer"
-F 6 "311-1.0KGRCT-ND" H 7075 1825 50  0001 C CNN "Supplier:Digikey"
+F 6 "311-10.0KHRCT-ND" H 7075 1825 50  0001 C CNN "Supplier:Digikey"
 	1    7075 1825
 	0    1    1    0
